File: LED-Cube_MK3.sch (KiCad schematic (older format))
At the start: 31 parts, among them Q1 2N7002, Q2 2N7002, Q3 2N7002, Q4 2N7002, SW1 SW_Push, SW2 SW_Push, U1 74HC595, U2 74HC595, U3 LED_Cube_5mm_4x4x4

Commit message: change led spacing to 15mm and add arduino 3d model
Signed-off-by: Thomas Schmid <tom@binary-kitchen.de>
Connections:
- net mode_sw: now reaches A1.7 (D4), SW2.2
- net QH*: now reaches U1.9 (QH'), U2.14 (SER)
- net at R5.1: now also U3.1 (LED_13); no longer U3.4 (LED_01)
- net at R6.1: now also U3.2 (LED_09); no longer U3.5 (LED_02)
- net at R7.1: now also U3.3 (LED_05); no longer U3.12 (LED_03)
- net at R8.1: now also U3.4 (LED_01); no longer U3.13 (LED_04)
- net at R9.1: now also U3.5 (LED_02); no longer U3.3 (LED_05)
- net at R11.1: now also U3.7 (LED_10); no longer U3.11 (LED_07)
- net at R12.1: now also U3.8 (LED_14); no longer U3.14 (LED_08)
- net at R13.1: now also U3.9 (LED_15); no longer U3.2 (LED_09)
- net at R14.1: now also U3.10 (LED_11); no longer U3.7 (LED_10)
- net at R15.1: now also U3.11 (LED_07); no longer U3.10 (LED_11)
- net at R16.1: now also U3.12 (LED_03); no longer U3.15 (LED_12)
- net at R17.1: now also U3.13 (LED_04); no longer U3.1 (LED_13)
- net at R18.1: now also U3.14 (LED_08); no longer U3.8 (LED_14)
- net at R19.1: now also U3.15 (LED_12); no longer U3.9 (LED_15)
- net LED01 renamed LED_1
- net LED_1: now also R8.2; no longer R5.2
- net LED02 renamed LED_2
- net LED_2: now also R9.2; no longer R6.2
- net LED03 renamed LED_3
- net LED_3: now also R16.2; no longer R7.2
- net LED04 renamed LED_4
- net LED_4: now also R17.2; no longer R8.2
- net LED05 renamed LED_5
- net LED_5: now also R7.2; no longer R9.2
- net LED06 renamed LED_6
- net LED07 renamed LED_10
- net LED_10: now also U2.1 (QB); no longer U1.6 (QG)
- net LED08 renamed LED_14
- net LED_14: now also U2.5 (QF); no longer U1.7 (QH)
- net LED09 renamed LED_15
- net LED_15: now also U2.6 (QG); no longer U2.15 (QA)
- net LED10 renamed LED_11
- net LED_11: now also U2.2 (QC); no longer U2.1 (QB)
- net LED11 renamed LED_7
- net LED_7: now also U1.6 (QG); no longer U2.2 (QC)
- net LED12 renamed LED_12
- net LED_12: now also R19.2; no longer R16.2
- net LED13 renamed LED_13
- net LED_13: now also R5.2; no longer R17.2
- net LED14 renamed LED_8
- net LED_8: now also U1.7 (QH); no longer U2.5 (QF)
- removed net LED15: R19.2, U2.6 (QG)
- net LED16 renamed LED_16
- new net LED_9: R6.2, U2.15 (QA)
Other:
- moved on the sheet: R10, R11, R12, R13, R14, R15, R16, R17, R18, R19, R20, R5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

Commit message: Add missing part values
Signed-off-by: Thomas Schmid <thomas.schmid111@web.de>
Parts:
- R1, R2, R3, R4: value R -> 1k
- R10, R11, R12, R13, R14, R15, R16, R17, R18, R19, R20, R5, R6, R7, R8, R9: value R -> 52
Changed lines of the file:
@@
 P 10250 3250
 F 0 "R5" V 10043 3250 50  0000 C CNN
-F 1 "R" V 10134 3250 50  0000 C CNN
+F 1 "52" V 10134 3250 50  0000 C CNN
 F 2 "Resistor_SMD:R_0805_2012Metric_Pad1.15x1.40mm_HandSolder" V 10180 3250 50  0001 C CNN
 F 3 "~" H 10250 3250 50  0001 C CNN
@@
 P 10250 2650
 F 0 "R6" V 10043 2650 50  0000 C CNN
-F 1 "R" V 10134 2650 50  0000 C CNN
+F 1 "52" V 10134 2650 50  0000 C CNN
 F 2 "Resistor_SMD:R_0805_2012Metric_Pad1.15x1.40mm_HandSolder" V 10180 2650 50  0001 C CNN
 F 3 "~" H 10250 2650 50  0001 C CNN
@@
 P 10250 2050
 F 0 "R7" V 10043 2050 50  0000 C CNN
-F 1 "R" V 10134 2050 50  0000 C CNN
+F 1 "52" V 10134 2050 50  0000 C CNN
 F 2 "Resistor_SMD:R_0805_2012Metric_Pad1.15x1.40mm_HandSolder" V 10180 2050 50  0001 C CNN
 F 3 "~" H 10250 2050 50  0001 C CNN
@@
 P 10250 1450
 F 0 "R8" V 10043 1450 50  0000 C CNN
-F 1 "R" V 10134 1450 50  0000 C CNN
+F 1 "52" V 10134 1450 50  0000 C CNN
 F 2 "Resistor_SMD:R_0805_2012Metric_Pad1.15x1.40mm_HandSolder" V 10180 1450 50  0001 C CNN
 F 3 "~" H 10250 1450 50  0001 C CNN
@@
 P 10250 1600
 F 0 "R9" V 10043 1600 50  0000 C CNN
-F 1 "R" V 10134 1600 50  0000 C CNN
+F 1 "52" V 10134 1600 50  0000 C CNN
 F 2 "Resistor_SMD:R_0805_2012Metric_Pad1.15x1.40mm_HandSolder" V 10180 1600 50  0001 C CNN
 F 3 "~" H 10250 1600 50  0001 C CNN
@@
 P 10250 2200
 F 0 "R10" V 10043 2200 50  0000 C CNN
-F 1 "R" V 10134 2200 50  0000 C CNN
+F 1 "52" V 10134 2200 50  0000 C CNN
 F 2 "Resistor_SMD:R_0805_2012Metric_Pad1.15x1.40mm_HandSolder" V 10180 2200 50  0001 C CNN
 F 3 "~" H 10250 2200 50  0001 C CNN
@@
 P 10250 2800
 F 0 "R11" V 10043 2800 50  0000 C CNN
-F 1 "R" V 10134 2800 50  0000 C CNN
+F 1 "52" V 10134 2800 50  0000 C CNN
 F 2 "Resistor_SMD:R_0805_2012Metric_Pad1.15x1.40mm_HandSolder" V 10180 2800 50  0001 C CNN
 F 3 "~" H 10250 2800 50  0001 C CNN
@@
 P 10250 3400
 F 0 "R12" V 10043 3400 50  0000 C CNN
-F 1 "R" V 10134 3400 50  0000 C CNN
+F 1 "52" V 10134 3400 50  0000 C CNN
 F 2 "Resistor_SMD:R_0805_2012Metric_Pad1.15x1.40mm_HandSolder" V 10180 3400 50  0001 C CNN
 F 3 "~" H 10250 3400 50  0001 C CNN
@@
 P 10250 3550
 F 0 "R13" V 10043 3550 50  0000 C CNN
-F 1 "R" V 10134 3550 50  0000 C CNN
+F 1 "52" V 10134 3550 50  0000 C CNN
 F 2 "Resistor_SMD:R_0805_2012Metric_Pad1.15x1.40mm_HandSolder" V 10180 3550 50  0001 C CNN
 F 3 "~" H 10250 3550 50  0001 C CNN
@@
 P 10250 2950
 F 0 "R14" V 10043 2950 50  0000 C CNN
-F 1 "R" V 10134 2950 50  0000 C CNN
+F 1 "52" V 10134 2950 50  0000 C CNN
 F 2 "Resistor_SMD:R_0805_2012Metric_Pad1.15x1.40mm_HandSolder" V 10180 2950 50  0001 C CNN
 F 3 "~" H 10250 2950 50  0001 C CNN
@@
 P 10250 2350
 F 0 "R15" V 10043 2350 50  0000 C CNN
-F 1 "R" V 10134 2350 50  0000 C CNN
+F 1 "52" V 10134 2350 50  0000 C CNN
 F 2 "Resistor_SMD:R_0805_2012Metric_Pad1.15x1.40mm_HandSolder" V 10180 2350 50  0001 C CNN
 F 3 "~" H 10250 2350 50  0001 C CNN
@@
 P 10250 1750
 F 0 "R16" V 10043 1750 50  0000 C CNN
-F 1 "R" V 10134 1750 50  0000 C CNN
+F 1 "52" V 10134 1750 50  0000 C CNN
 F 2 "Resistor_SMD:R_0805_2012Metric_Pad1.15x1.40mm_HandSolder" V 10180 1750 50  0001 C CNN
 F 3 "~" H 10250 1750 50  0001 C CNN
@@
 P 10250 1900
 F 0 "R17" V 10043 1900 50  0000 C CNN
-F 1 "R" V 10134 1900 50  0000 C CNN
+F 1 "52" V 10134 1900 50  0000 C CNN
 F 2 "Resistor_SMD:R_0805_2012Metric_Pad1.15x1.40mm_HandSolder" V 10180 1900 50  0001 C CNN
 F 3 "~" H 10250 1900 50  0001 C CNN
@@
 P 10250 2500
 F 0 "R18" V 10043 2500 50  0000 C CNN
-F 1 "R" V 10134 2500 50  0000 C CNN
+F 1 "52" V 10134 2500 50  0000 C CNN
 F 2 "Resistor_SMD:R_0805_2012Metric_Pad1.15x1.40mm_HandSolder" V 10180 2500 50  0001 C CNN
 F 3 "~" H 10250 2500 50  0001 C CNN
@@
 P 10250 3100
 F 0 "R19" V 10043 3100 50  0000 C CNN
-F 1 "R" V 10134 3100 50  0000 C CNN
+F 1 "52" V 10134 3100 50  0000 C CNN
 F 2 "Resistor_SMD:R_0805_2012Metric_Pad1.15x1.40mm_HandSolder" V 10180 3100 50  0001 C CNN
 F 3 "~" H 10250 3100 50  0001 C CNN
@@
 P 10250 3700
 F 0 "R20" V 10043 3700 50  0000 C CNN
-F 1 "R" V 10134 3700 50  0000 C CNN
+F 1 "52" V 10134 3700 50  0000 C CNN
 F 2 "Resistor_SMD:R_0805_2012Metric_Pad1.15x1.40mm_HandSolder" V 10180 3700 50  0001 C CNN
 F 3 "~" H 10250 3700 50  0001 C CNN
@@
 P 9000 5250
 F 0 "R3" V 8793 5250 50  0000 C CNN
-F 1 "R" V 8884 5250 50  0000 C CNN
+F 1 "1k" V 8884 5250 50  0000 C CNN
 F 2 "Resistor_SMD:R_0805_2012Metric_Pad1.15x1.40mm_HandSolder" V 8930 5250 50  0001 C CNN
 F 3 "~" H 9000 5250 50  0001 C CNN
@@
 P 10150 5250
 F 0 "R4" V 9943 5250 50  0000 C CNN
-F 1 "R" V 10034 5250 50  0000 C CNN
+F 1 "1k" V 10034 5250 50  0000 C CNN
 F 2 "Resistor_SMD:R_0805_2012Metric_Pad1.15x1.40mm_HandSolder" V 10080 5250 50  0001 C CNN
 F 3 "~" H 10150 5250 50  0001 C CNN
@@
 P 6800 5250
 F 0 "R1" V 6593 5250 50  0000 C CNN
-F 1 "R" V 6684 5250 50  0000 C CNN
+F 1 "1k" V 6684 5250 50  0000 C CNN
 F 2 "Resistor_SMD:R_0805_2012Metric_Pad1.15x1.40mm_HandSolder" V 6730 5250 50  0001 C CNN
 F 3 "~" H 6800 5250 50  0001 C CNN
@@
 P 7900 5250
 F 0 "R2" V 7693 5250 50  0000 C CNN
-F 1 "R" V 7784 5250 50  0000 C CNN
+F 1 "1k" V 7784 5250 50  0000 C CNN
 F 2 "Resistor_SMD:R_0805_2012Metric_Pad1.15x1.40mm_HandSolder" V 7830 5250 50  0001 C CNN
 F 3 "~" H 7900 5250 50  0001 C CNN
